Commit message: force a nous

File: src/turtlebot3_descriptions/urdf/turtlebot3_burger_d435i.urdf (robot description, URDF)
Before this commit: robot turtlebot3_burger, 10 links, 9 joints
Links:
- added link support_cameras_a_link; collision box size=0.09 0.03 0.015; visual mesh filename=package://turtlebot3_descriptions/meshes/sensors/support_ca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 scale=0.001 0.001 0.001
- added link support_cameras_b_link; collision box size=0.09 0.025 0.015; visual mesh filename=package://turtlebot3_descriptions/meshes/sensors/support_ca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 scale=0.001 0.001 0.001
Joints:
- added joint support_cameras_a_joint: type fixed, parent base_link, child support_cameras_a_link, origin xyz=0.023 0 0.101 rpy=0 0 0
- added joint support_cameras_b_joint: type fixed, parent support_cameras_a_link, child support_cameras_b_link, origin xyz=0.0435 0 0 rpy=0 -1.57 0
- joint joint_d435i_camera: origin xyz=0.047 0.0 0.11 rpy=0.0 0.0 0.0 -> xyz=0.0613 0.0 0.028 rpy=0 0 0; parent base_link -> support_cameras_a_link
- joint joint_d435i_color_optical_frame: origin xyz=0.0 0.0 0.0 rpy=-1.5708 0.0 -1.5708 -> xyz=0.1 0.0 0.0 rpy=0 0 0
- joint joint_d435i_depth_optical_frame: origin xyz=0.0 0.0 0.0 rpy=-1.5708 0.0 -1.5708 -> xyz=0.0 0.0 0.0 rpy=0 0 0

File: src/turtlebot3_descriptions/urdf/turtlebot3_burger_gripper.urdf (robot description, URDF)
Before this commit: robot turtlebot3_burger, 11 links, 10 joints
Links:
- added link counterweight, mass 0.3
- added link oak_d_pro_camera, mass 0.09100000; collision box size=0.1 0.03 0.02; visual mesh filename=package://turtlebot3_descriptions/meshes/sensors/OAK-D-PRO.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 scale=1.0 1.0 1.0
- added link oak_d_pro_color_optical_frame
- added link oak_d_pro_depth_optical_frame
- added link support_cameras_a_link; collision box size=0.09 0.03 0.015; visual mesh filename=package://turtlebot3_descriptions/meshes/sensors/support_ca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 scale=0.001 0.001 0.001
- added link support_cameras_b_link; collision box size=0.09 0.025 0.015; visual mesh filename=package://turtlebot3_descriptions/meshes/sensors/support_ca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 scale=0.001 0.001 0.001
- link base_gripper: mass 0.06 -> 0.07390000; geometry collision box size=0.055 0.055 0.06; visual mesh filename=package://turtlebot3_descriptions/meshes/actuators/gripper/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 scale=0.001 0.001 0.001
Joints:
- added joint joint_counterweight: type fixed, parent base_link, child counterweight, origin xyz=-0.12 0.0 0.0 rpy=0 0 0
- added joint joint_oak_d_pro_camera: type fixed, parent support_cameras_b_link, child oak_d_pro_camera, origin xyz=0.0315 -0.0015 -0.03 rpy=3.14 0 1.57
- added joint joint_oak_d_pro_color_optical_frame: type fixed, parent oak_d_pro_camera, child oak_d_pro_color_optical_frame, origin xyz=0.0 0.0 0.0 rpy=0 0 0
- added joint joint_oak_d_pro_depth_optical_frame: type fixed, parent oak_d_pro_camera, child oak_d_pro_depth_optical_frame, origin xyz=0.0 0.0 0.0 rpy=-1.57 -1.57 0
- added joint support_cameras_a_joint: type fixed, parent base_link, child support_cameras_a_link, origin xyz=0.023 0 0.101 rpy=0 0 0
- added joint support_cameras_b_joint: type fixed, parent support_cameras_a_link, child support_cameras_b_link, origin xyz=0.0435 0 0 rpy=0 -1.57 0
- joint gripper_base_joint: origin xyz=0.052 0.0025 0.04 rpy=0 0 0 -> xyz=0.023 0.0025 0.08 rpy=0 0 -1.57
- joint gripper_tilt_joint: origin xyz=0 0.002 0 rpy=0 0 0 -> xyz=-0.0005 0.0335 -0.033 rpy=0 0 1.57

File: src/turtlebot3_descriptions/urdf/turtlebot3_burger_oak_d_pro.urdf (robot description, URDF)
Before this commit: robot turtlebot3_burger, 10 links, 9 joints
Links:
- added link support_cameras_a_link; collision box size=0.09 0.03 0.015; visual mesh filename=package://turtlebot3_descriptions/meshes/sensors/support_ca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 scale=0.001 0.001 0.001
- added link support_cameras_b_link; collision box size=0.09 0.025 0.015; visual mesh filename=package://turtlebot3_descriptions/meshes/sensors/support_ca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 scale=0.001 0.001 0.001
Joints:
- added joint support_cameras_a_joint: type fixed, parent base_link, child support_cameras_a_link, origin xyz=0.023 0 0.101 rpy=0 0 0
- added joint support_cameras_b_joint: type fixed, parent support_cameras_a_link, child support_cameras_b_link, origin xyz=0.0435 0 0 rpy=0 -1.57 0
- joint joint_oak_d_pro_camera: origin xyz=0.065 0.0 0.11 rpy=1.57 0.0 1.57 -> xyz=0.0315 -0.0015 -0.026 rpy=3.14 0 1.57; parent base_link -> support_cameras_b_link
- joint joint_oak_d_pro_color_optical_frame: origin xyz=0.0 0.0 0.0 rpy=-1.5708 0.0 -1.5708 -> xyz=0.0 0.0 0.0 rpy=0 0 0
- joint joint_oak_d_pro_depth_optical_frame: origin xyz=0.0 0.0 0.0 rpy=-1.5708 0.0 -1.5708 -> xyz=0.0 0.0 0.0 rpy=-1.57 -1.57 0

File: src/turtlebot3_descriptions/urdf/turtlebot3_burger_pi_cam.urdf (robot description, URDF)
Before this commit: robot turtlebot3_burger, 9 links, 8 joints
Links:
- added link support_cameras_a_link; collision box size=0.09 0.03 0.015; visual mesh filename=package://turtlebot3_descriptions/meshes/sensors/support_ca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 scale=0.001 0.001 0.001
- added link support_cameras_b_link; collision box size=0.09 0.025 0.015; visual mesh filename=package://turtlebot3_descriptions/meshes/sensors/support_ca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 scale=0.001 0.001 0.001
Joints:
- added joint support_cameras_a_joint: type fixed, parent base_link, child support_cameras_a_link, origin xyz=0.023 0 0.101 rpy=0 0 0
- added joint support_cameras_b_joint: type fixed, parent support_cameras_a_link, child support_cameras_b_link, origin xyz=0.0435 0 0 rpy=0 -1.57 0
- joint joint_pi_camera: origin xyz=0.05 0.0 0.11 rpy=0 0 3.14 -> xyz=0.0606 -0.0 0.018 rpy=3.14 0 3.14; parent base_link -> support_cameras_a_link
